Commit message: [dhairya]: add slam_bot urdf, launch files and lidar support, rgb camera still left

File: Software/Ros/src/virtual_lab/urdf/mogi_bot.urdf (robot description, URDF)
Before this commit: robot mogi_bot, 4 links, 3 joints
Links:
- link base_link: geometry collision box size=.4 .2 .1; collision sphere radius=0.0499
- link left_wheel: geometry collision cylinder length=.05 radius=.1; visual mesh filename=package://virtual_lab/meshes/wheel.dae
- link right_wheel: geometry collision cylinder length=.05 radius=.1; visual mesh filename=package://virtual_lab/meshes/wheel.dae

File: Software/Ros/src/virtual_lab/urdf/slam_bot.urdf (robot description, URDF)
Before this commit: robot slam_bot, 7 links, 6 joints
Links:
- added link base_footprint
Joints:
- added joint base_footprint_joint: type fixed, parent base_footprint, child base_link, origin xyz=0 0 0 rpy=0 0 0
- joint bk_left_wheel_joint: axis 0 1 0 -> 0 0 -1; limit (none) -> effort=2.94 velocity=4.712; origin xyz=0.73816 -1.2653 0.82211 rpy=1.5708 1.379 1.5708 -> xyz=-0.065591 0.1053 0.017276 rpy=-1.5708 0 0
- joint bk_right_wheel_joint: axis 0 1 0 -> 0 0 1; limit (none) -> effort=2.94 velocity=4.712; origin xyz=0.52756 -1.2653 0.82211 rpy=-1.5708 1.379 1.5708 -> xyz=-0.065606 -0.1053 0.017279 rpy=-1.5708 0 0
- joint camera_joint: origin xyz=0.63286 -1.3938 0.89301 rpy=1.1384 0 0 -> xyz=0.06293 0 0.088176 rpy=0 -0.43241 0
- joint fr_left_wheel_joint: axis 0 1 0 -> 0 0 -1; limit (none) -> effort=2.94 velocity=4.712; origin xyz=0.73816 -1.3964 0.82211 rpy=-1.5708 1.379 -1.5708 -> xyz=0.065506 0.1053 0.017279 rpy=-1.5708 0 0
- joint fr_right_wheel_joint: axis 0 1 0 -> 0 0 1; limit (none) -> effort=2.94 velocity=4.712; origin xyz=0.52756 -1.3964 0.82211 rpy=1.5708 1.379 -1.5708 -> xyz=0.065492 -0.1053 0.017276 rpy=-1.5708 0 0
- joint lidar_joint: origin xyz=0.63307 -1.3458 0.93783 rpy=1.5708 0 0 -> xyz=0.01495 0.00020855 0.133 rpy=0 0 0
