Commit message: [dhairya]: fixed urdf & world models path issue, add support for rgb camera, imu still left

File: Software/Ros/src/virtual_lab/urdf/slam_bot.urdf (robot description, URDF)
Before this commit: robot virtual_lab, 8 links, 7 joints
Links:
- added link camera_link_optical
Joints:
- added joint camera_optical_joint: type fixed, parent camera_link, child camera_link_optical, origin xyz=0 0 0 rpy=-1.5707 0 -1.5707
- joint camera_joint: axis 0 0 0 -> (none)
- joint lidar_joint: axis 0 0 0 -> (none)
